Commit message: Hackathon Roboter gefixt und Friedberd hinzugefügt

File: urdf/hackathon_robot.urdf (robot description, URDF)
Before this commit: robot my_robot, 6 links, 5 joints
Links:
- link base_link: geometry collision mesh filename=file:///home/andi/project/ros2_workspace/src/self_driving_b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 scale=0.002 0.002 0.002; visual mesh filename=file:///home/andi/project/ros2_workspace/src/self_driving_b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 scale=0.002 0.002 0.002
- link left_front_wheel: mass 0.1 -> 0.05; geometry collision cylinder length=0.05 radius=0.032; visual cylinder length=0.05 radius=0.07
- link left_wheel: geometry collision cylinder length=0.05 radius=0.07; visual cylinder length=0.05 radius=0.07
- link right_front_wheel: geometry collision cylinder length=0.05 radius=0.07; visual cylinder length=0.05 radius=0.07
- link right_wheel: geometry collision cylinder length=0.05 radius=0.07; visual cylinder length=0.05 radius=0.07
Joints:
- joint left_front_wheel_joint: limit (none) -> lower=-3.14 upper=3.14 effort=0.0 velocity=100.0; origin xyz=0.070 -0.060 0 rpy=1.5708 0 0 -> xyz=0.12 0.111 0.065 rpy=1.5708 0 0
- joint left_wheel_joint: origin xyz=-0.070 -0.062 0 rpy=1.5708 0 0 -> xyz=-0.12 0.111 0.065 rpy=1.5708 0 0
- joint right_front_wheel_joint: limit (none) -> lower=-3.14 upper=3.14 effort=0.0 velocity=100.0; origin xyz=0.070 0.060 0 rpy=1.5708 0 0 -> xyz=0.12 -0.111 0.065 rpy=1.5708 0 0
- joint right_wheel_joint: origin xyz=-0.070 0.062 0 rpy=1.5708 0 0 -> xyz=-0.12 -0.111 0.065 rpy=1.5708 0 0
