Commit message: Verzeichnis in urdf File gefixt

File: urdf/friedbert.urdf (robot description, URDF)
Before this commit: robot my_robot, 12 links, 11 joints
Links:
- link base_link: geometry collision mesh filename=file://$(find self_driving_bot)/meshes/torso.stl scale=0.002 0.002 0.002; visual mesh filename=file://$(find self_driving_bot)/meshes/torso.stl scale=0.002 0.002 0.002
- link head: geometry collision mesh filename=file://$(find self_driving_bot)/head.stl scale=0.002 0.002 0.002; visual mesh filename=file://$(find self_driving_bot)/meshes/head.stl scale=0.002 0.002 0.002
- link left_lower_arm: geometry collision mesh filename=file://$(find self_driving_bot)/meshes/left_lower_arm.stl scale=0.002 0.002 0.002; visual mesh filename=file://$(find self_driving_bot)/meshes/left_lower_arm.stl scale=0.002 0.002 0.002
- link left_upper_arm: geometry collision mesh filename=file://$(find self_driving_bot)/meshes/left_upper_arm.stl scale=0.002 0.002 0.002; visual mesh filename=file://$(find self_driving_bot)/meshes/left_upper_arm.stl scale=0.002 0.002 0.002
- link neck: geometry collision mesh filename=file://$(find self_driving_bot)/meshes/neck.stl scale=0.002 0.002 0.002; visual mesh filename=file://$(find self_driving_bot)/meshes/neck.stl scale=0.002 0.002 0.002
- link right_lower_arm: geometry collision mesh filename=file://$(find self_driving_bot)/meshes/right_lower_arm.stl scale=0.002 0.002 0.002; visual mesh filename=file://$(find self_driving_bot)/meshes/right_lower_arm.stl scale=0.002 0.002 0.002
- link right_upper_arm: geometry collision mesh filename=file://$(find self_driving_bot)/meshes/right_upper_arm.stl scale=0.002 0.002 0.002; visual mesh filename=file://$(find self_driving_bot)/meshes/right_upper_arm.stl scale=0.002 0.002 0.002

File: urdf/hackathon_robot.urdf (robot description, URDF)
Before this commit: robot my_robot, 6 links, 5 joints
Links:
- link base_link: geometry collision mesh filename=file://$(find self_driving_bot)/meshes/robot.stl scale=0.002 0.002 0.002; visual mesh filename=file://$(find self_driving_bot)/meshes/robot.stl scale=0.002 0.002 0.002

Commit message: Kameras in den Roboter eingebaut

File: urdf/friedbert.urdf (robot description, URDF)
Before this commit: robot my_robot, 12 links, 11 joints
Links:
- added link left_eye; collision cylinder length=0.02 radius=0.01; visual cylinder length=0.02 radius=0.012
- added link right_eye; collision cylinder length=0.02 radius=0.01; visual cylinder length=0.02 radius=0.012
Joints:
- added joint left_eye_joint: type fixed, parent head, child left_eye, origin xyz=0.07 0.05 0.04 rpy=0 0 0
- added joint right_eye_joint: type fixed, parent head, child right_eye, origin xyz=0.07 -0.05 0.04 rpy=0 0 0
