Commit message: test_zone world added

File: urdf/ikea_table.urdf (robot description, URDF)
Before this commit: robot ikea_table, 10 links, 9 joints
Links:
- link roll_front_left: geometry collision mesh filename=file:///home/andi/ros2/ros2_workspace/install/self_driving_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 scale=1 1 1; visual mesh filename=file:///home/andi/ros2/ros2_workspace/install/self_driving_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 scale=1 1 1
- link roll_front_right: geometry collision mesh filename=file:///home/andi/ros2/ros2_workspace/install/self_driving_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 scale=1 1 1; visual mesh filename=file:///home/andi/ros2/ros2_workspace/install/self_driving_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 scale=1 1 1

Commit message: test

File: urdf/ikea_table.urdf (robot description, URDF)
Before this commit: robot ikea_table, 12 links, 11 joints
Links:
- link chassis: geometry collision mesh filename=file:///home/andi/ros2_workspace/install/self_driving_bot/s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 scale=1 1 1; visual mesh filename=file:///home/andi/ros2_workspace/install/self_driving_bot/s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 scale=1 1 1
- link roll_front_left: geometry collision mesh filename=file:///home/andi/ros2_workspace/install/self_driving_bot/s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 scale=1 1 1; visual mesh filename=file:///home/andi/ros2_workspace/install/self_driving_bot/s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 scale=1 1 1
- link roll_front_right: geometry collision mesh filename=file:///home/andi/ros2_workspace/install/self_driving_bot/s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 scale=1 1 1; visual mesh filename=file:///home/andi/ros2_workspace/install/self_driving_bot/s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 scale=1 1 1

Commit message: funktionierender Stand

File: urdf/ikea_table.urdf (robot description, URDF)
Before this commit: robot ikea_table, 12 links, 11 joints
Links:
- link chassis: geometry collision mesh filename=file:///home/andi/project/ros2_workspace/install/self_drivi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 scale=1 1 1; visual mesh filename=file:///home/andi/project/ros2_workspace/install/self_drivi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 scale=1 1 1
- link roll_front_left: geometry collision mesh filename=file:///home/andi/project/ros2_workspace/install/self_drivi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 scale=1 1 1; visual mesh filename=file:///home/andi/project/ros2_workspace/install/self_drivi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 scale=1 1 1
- link roll_front_right: geometry collision mesh filename=file:///home/andi/project/ros2_workspace/install/self_drivi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 scale=1 1 1; visual mesh filename=file:///home/andi/project/ros2_workspace/install/self_drivi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 scale=1 1 1

Commit message: urdf file in physical navigation hinzugefügt

File: urdf/ikea_table.urdf (robot description, URDF)
Before this commit: robot ikea_table, 12 links, 11 joints
Links:
- removed link rplidar_link
- added link base_laser, mass 0.1; collision cylinder length=0.02 radius=0.065; visual cylinder length=0.02 radius=0.065
- link chassis: geometry collision mesh filename=file:///home/andi/ros2_workspace/install/self_driving_bot/s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 scale=1 1 1; visual mesh filename=file:///home/andi/ros2_workspace/install/self_driving_bot/s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 scale=1 1 1
- link roll_front_left: geometry collision mesh filename=file:///home/andi/ros2_workspace/install/self_driving_bot/s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 scale=1 1 1; visual mesh filename=file:///home/andi/ros2_workspace/install/self_driving_bot/s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 scale=1 1 1
- link roll_front_right: geometry collision mesh filename=file:///home/andi/ros2_workspace/install/self_driving_bot/s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 scale=1 1 1; visual mesh filename=file:///home/andi/ros2_workspace/install/self_driving_bot/s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 scale=1 1 1
Joints:
- joint base_footprint_joint: child base_footprint -> base_link; parent base_link -> base_footprint
- joint lidar_joint: child rplidar_link -> base_laser
